Commit message: Improve fingray fingers

File: blender_models/tri_finray_gripper/finray_finger_assembly_box_collision_2.urdf (robot description, URDF)
Before this commit: robot tri_finray_gripper, 5 links, 4 joints
Links:
- link finger_holder_left: geometry collision box size=0.04 0.06979999499999999 0.038
- link finger_holder_right: geometry collision box size=0.04 0.06979999499999999 0.038
- link soft_finger_left: geometry collision box size=0.039999924 0.025800001000000003 0.123364487; visual mesh filename=package://blender_models/tri_finray_gripper/meshes/one_piec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 scale=1 1 1
- link soft_finger_right: geometry collision box size=0.039999924 0.025800001000000003 0.123364487; visual mesh filename=package://blender_models/tri_finray_gripper/meshes/one_piec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 scale=1 1 1
